File: LoRa/LoRa.sch (EAGLE design)
At the start: 8 parts, among them J1 UP2-AH-1-TH, U1 RFM69HCW, U3 AP2112K-3.3, X1 uFL/SMA

Commit message: More stuff added
Parts:
- added IC1: FT232RL, ftdichip:FT232RL
- added IC2: STM32L072CZT7, STM32L072CZT7:STM32L072CZT7
Changed lines of the file:
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@@
 <part name="+5V1" library="microbuilder" deviceset="VIN" device=""/>
 <part name="U$1" library="microbuilder" deviceset="GND" device=""/>
+<part name="IC1" library="ftdichip" library_urn="urn:adsk.eagle:library:231" deviceset="FT232R" device="L" package3d_urn="urn:adsk.eagle:package:14013/1"/>
+<part name="IC2" library="STM32L072CZT7" deviceset="STM32L072CZT7" device=""/>
 </parts>
 <sheets>
@@
 <text x="53.34" y="241.3" size="1.778" layer="91">LoRa Module</text>
 <text x="154.94" y="233.68" size="1.778" layer="91">Linear Regulator</text>
-<text x="40.64" y="170.18" size="1.778" layer="91">PULL UP CS and RST using 100k?</text>
+<text x="22.86" y="187.96" size="1.778" layer="91">PULL UP CS and RST using 100k?</text>
 </plain>
 <instances>
@@
 <instance part="+5V1" gate="G$1" x="226.06" y="233.68"/>
 <instance part="U$1" gate="G$1" x="269.24" y="215.9"/>
+<instance part="IC1" gate="1" x="58.42" y="91.44"/>
+<instance part="IC2" gate="G$1" x="175.26" y="78.74"/>
 </instances>
 <busses>
