File: LoRa/LoRa.brd (EAGLE design)
At the start: 67 x 20.3 mm, 8 parts, among them J1 UP2-AH-1-TH, U1 RFM69HCW, U3 AP2112K-3.3, X1 uFL/SMA

Commit message: More stuff added
Parts:
- added IC1: FT232RL, ftdichip:SSOP28
- added IC2: STM32L072CZT7, STM32L072CZT7:QFP50P900X900X160-48N
Connections:
- new net VCC: IC1.20
- new net VCCIO: IC1.4
- net GND: now also IC1.18, IC1.21, IC1.25, IC1.7
Changed lines of the file:
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@@
 <setting verticaltext="up"/>
 </settings>
-<grid distance="10" unitdist="mil" unit="mil" style="lines" multiple="1" display="yes" altdistance="5" altunitdist="mil" altunit="mil"/>
+<grid distance="50" unitdist="mil" unit="mil" style="lines" multiple="1" display="yes" altdistance="5" altunitdist="mil" altunit="mil"/>
 <layers>
 <layer number="1" name="Top" color="4" fill="1" visible="yes" active="yes"/>
@@
 <attribute name="RS_PRICE-STOCK" value="" x="81.534" y="10.414" size="1.778" layer="27" rot="R90" display="off"/>
 </element>
+<element name="IC1" library="ftdichip" library_urn="urn:adsk.eagle:library:231" package="SSOP28" package3d_urn="urn:adsk.eagle:package:14013/1" value="FT232RL" x="54.864" y="7.112" rot="R270">
+<attribute name="MF" value="" x="54.864" y="7.112" size="1.778" layer="27" rot="R270" display="off"/>
+<attribute name="MPN" value="FT232RL" x="54.864" y="7.112" size="1.778" layer="27" rot="R270" display="off"/>
+<attribute name="OC_FARNELL" value="1146032" x="54.864" y="7.112" size="1.778" layer="27" rot="R270" display="off"/>
+<attribute name="OC_NEWARK" value="91K9918" x="54.864" y="7.112" size="1.778" layer="27" rot="R270" display="off"/>
+<attribute name="POPULARITY" value="14" x="54.864" y="7.112" size="1.778" layer="27" rot="R270" display="off"/>
+</element>
+<element name="IC2" library="STM32L072CZT7" package="QFP50P900X900X160-48N" value="STM32L072CZT7" x="37.846" y="9.906">
+<attribute name="DESCRIPTION" value="ARM Microcontrollers - MCU 16/32-BITS MICROS" x="37.846" y="9.906" size="1.778" layer="27" display="off"/>
+<attribute name="HEIGHT" value="1.6mm" x="37.846" y="9.906" size="1.778" layer="27" display="off"/>
+<attribute name="MANUFACTURER_NAME" value="STMicroelectronics" x="37.846" y="9.906" size="1.778" layer="27" display="off"/>
+<attribute name="MANUFACTURER_PART_NUMBER" value="STM32L072CZT7" x="37.846" y="9.906" size="1.778" layer="27" display="off"/>
+<attribute name="MOUSER_PART_NUMBER" value="511-STM32L072CZT7" x="37.846" y="9.906" size="1.778" layer="27" display="off"/>
+<attribute name="MOUSER_PRICE-STOCK" value="https://www.mouser.com/Search/Refine.aspx?Keyword=511-STM32L072CZT7" x="37.846" y="9.906" size="1.778" layer="27" display="off"/>
+<attribute name="RS_PART_NUMBER" value="" x="37.846" y="9.906" size="1.778" layer="27" display="off"/>
+<attribute name="RS_PRICE-STOCK" value="" x="37.846" y="9.906" size="1.778" layer="27" display="off"/>
+</element>
 </elements>
 <signals>
@@
 <contactref element="C1" pad="2"/>
 <contactref element="J1" pad="4"/>
+<contactref element="IC1" pad="7"/>
+<contactref element="IC1" pad="25"/>
+<contactref element="IC1" pad="18"/>
+<contactref element="IC1" pad="21"/>
+<wire x1="56.896" y1="14.136" x2="54.6401" y2="16.764" width="0" layer="19" extent="1-1"/>
+<wire x1="61.634" y1="6.914" x2="56.896" y2="14.136" width="0" layer="19" extent="1-1"/>
+<wire x1="24.356" y1="16.144" x2="54.6401" y2="16.764" width="0" layer="19" extent="1-1"/>
+<wire x1="24.356" y1="2.144" x2="24.356" y2="16.144" width="0" layer="19" extent="1-1"/>
+<wire x1="8.156" y1="14.144" x2="24.356" y2="16.144" width="0" layer="19" extent="1-1"/>
+<wire x1="3.302" y1="12.7" x2="8.156" y2="14.144" width="0" layer="19" extent="1-1"/>
+<wire x1="3.302" y1="12.7" x2="3.302" y2="12.7" width="0" layer="19" extent="1-16"/>
+<wire x1="3.302" y1="17.78" x2="3.302" y2="12.7" width="0" layer="19" extent="1-1"/>
+<wire x1="3.302" y1="17.78" x2="3.302" y2="17.78" width="0" layer="19" extent="1-16"/>
+<wire x1="5.08" y1="6.262" x2="3.302" y2="12.7" width="0" layer="19" extent="1-1"/>
+<wire x1="58.489" y1="4.837" x2="5.08" y2="6.262" width="0" layer="19" extent="1-1"/>
+<wire x1="58.489" y1="6.787" x2="58.489" y2="4.837" width="0" layer="19" extent="1-1"/>
+<wire x1="58.489" y1="9.387" x2="58.489" y2="6.787" width="0" layer="19" extent="1-1"/>
+<wire x1="51.239" y1="7.437" x2="58.489" y2="6.787" width="0" layer="19" extent="1-1"/>
 </signal>
 <signal name="3.3V">
@@
 <contactref element="J1" pad="3"/>
 </signal>
+<signal name="VCC">
+<contactref element="IC1" pad="20"/>
+</signal>
+<signal name="VCCIO">
+<contactref element="IC1" pad="4"/>
+</signal>
 </signals>

Commit message: things and stuff
Parts:
- removed IC2: STM32L072CZT7, STM32L072CZT7:QFP50P900X900X160-48N
Changed lines of the file:
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@@
 <attribute name="POPULARITY" value="14" x="54.864" y="7.112" size="1.778" layer="27" rot="R270" display="off"/>
-</element>
-<element name="IC2" library="STM32L072CZT7" package="QFP50P900X900X160-48N" value="STM32L072CZT7" x="37.846" y="9.906">
-<attribute name="DESCRIPTION" value="ARM Microcontrollers - MCU 16/32-BITS MICROS" x="37.846" y="9.906" size="1.778" layer="27" display="off"/>
-<attribute name="HEIGHT" value="1.6mm" x="37.846" y="9.906" size="1.778" layer="27" display="off"/>
-<attribute name="MANUFACTURER_NAME" value="STMicroelectronics" x="37.846" y="9.906" size="1.778" layer="27" display="off"/>
-<attribute name="MANUFACTURER_PART_NUMBER" value="STM32L072CZT7" x="37.846" y="9.906" size="1.778" layer="27" display="off"/>
-<attribute name="MOUSER_PART_NUMBER" value="511-STM32L072CZT7" x="37.846" y="9.906" size="1.778" layer="27" display="off"/>
-<attribute name="MOUSER_PRICE-STOCK" value="https://www.mouser.com/Search/Refine.aspx?Keyword=511-STM32L072CZT7" x="37.846" y="9.906" size="1.778" layer="27" display="off"/>
-<attribute name="RS_PART_NUMBER" value="" x="37.846" y="9.906" size="1.778" layer="27" display="off"/>
-<attribute name="RS_PRICE-STOCK" value="" x="37.846" y="9.906" size="1.778" layer="27" display="off"/>
 </element>
 </elements>

Commit message: Stuff
Parts:
- removed IC1: FT232RL, ftdichip:SSOP28
- added C10, C11: 20pF, SparkFun-Capacitors:0603
- added C3, C5, C7: 1.0uF, SparkFun-Capacitors:0603
- added C4, C6: 0.1uF, SparkFun-Capacitors:0603
- added C8: 22uF, microbuilder:0805-NO
- added C9: 10uF, microbuilder:0805-NO
- added L1: 2.2uH/NRH2412T2R2MNGH, microbuilder:INDUCTOR_TAIYOYUDEN_NRH2412T
- added R2, R3, R4, R6: 10k, SparkFun-Resistors:0603
- added SV2: (no value), con-lsta:FE05-1
- added U2: RFM69HCW, microbuilder:RFMHCW_SMT
- added U4: BSS138, BSS138:SOT-23-3L
- added U5: LM3671MF-3.3/NOPB, microbuilder:SOT23-5
- added Y1: ECS-80-S-4X, ECS-80-S-4X:XTAL_ECS-80-S-4X
- C1: value 10uF -> 0.1uF
- U1: value RFM69HCW -> STM32L053C8T6; device microbuilder:RFMHCW_SMT -> STM32L053C8T6:QFP50P900X900X160-48N
- U3: value AP2112K-3.3 -> BSS138; device microbuilder:SOT23-5 -> BSS138:SOT-23-3L
- moved R1 37.3 mm to (23.4, 27.9), turned to 270 degrees
- moved C1 25.3 mm to (32.8, 7.37), flipped to the bottom
- moved C2 25.0 mm to (25.1, 22.1), flipped to the bottom, turned to 0 degrees
- moved U3 17.8 mm to (42.7, 2.54), turned to 270 degrees
- moved U1 15.8 mm to (32.0, 8.13), turned to 270 degrees
- moved J1 15.2 mm to (66.3, 10.2)
- moved X1 12.2 mm to (0.25, 3.05), flipped to the bottom, turned to 180 degrees
- moved JP2 12.2 mm to (5.59, 3.05)
Connections:
- removed net D_MINUS: J1.2
- removed net D_PLUS: J1.3
- removed net MISO: U1.10P
- removed net MOSI: U1.11P
- removed net SCK: U1.12P
- removed net VCC: IC1.20
- removed net VCCIO: IC1.4
- removed net VIN: C1.1, J1.1, R1.1, U3.1
- new net 5V: C9.1, J1.1, R1.1, R3.1, R6.1, U5.1
- new net EN: R1.2, U5.3
- new net NRST: SV2.1, U1.7
- new net OSC_IN: C11.1, U1.5, Y1.2
- new net OSC_OUT: C10.1, U1.6, Y1.1
- new net SPI1_MISO: U1.16, U2.10P
- new net SPI1_MOSI: U2.11P
- new net SPI1_SCK: U1.15, U2.12P
- new net SPI_MOSI: U1.17
- new net SWCLK: SV2.4, U1.37
- new net SWDIO: SV2.2, U1.34
- new net USB_DM_3V3: R4.1, U1.32, U4.2
- new net USB_DM_5V: J1.2, R6.2, U4.3
- new net USB_DP_3V3: R2.1, U1.33, U3.2
- new net USB_DP_5V: J1.3, R3.2, U3.3
- net 3.3V: now also C1.1, C3.1, C4.1, C5.1, C6.1, C7.1, C8.1, L1.2, R2.2, R4.2, SV2.5, U1.24, U1.36, U1.48, U1.9, U2.5P, U3.1, U4.1, U5.4; no longer U1.5P, U3.5
- net CS: now also U2.13P; no longer U1.13P
- net DIO0: now also U2.6P; no longer U1.6P
- net DIO1: now also U2.7P; no longer U1.7P
- net DIO2: now also U2.8P; no longer U1.8P
- net DIO3: now also U2.3P; no longer U1.3P
- net DIO4: now also U2.4P; no longer U1.4P
- net DIO5: now also U2.15P; no longer U1.15P
- net GND: now also C10.2, C11.2, C3.2, C4.2, C5.2, C6.2, C7.2, C8.2, C9.2, SV2.3, U1.23, U1.35, U1.47, U1.8, U2.16P, U2.2P, U2.9P, U5.2; no longer IC1.18, IC1.21, IC1.25, IC1.7, U1.16P, U1.2P, U1.9P, U3.2
- net N$1: now also U2.1P; no longer U1.1P
- net N$2: now also L1.1, U5.5; no longer R1.2, U3.3
- net RST: now also U2.14P; no longer U1.14P
Routing:
- net 3.3V: track 0.00 -> 30.6 mm, vias 0 -> 3
- net USB_DM_3V3: track 0.00 -> 17.0 mm, vias 0 -> 2
- net 5V: track 0.00 -> 13.6 mm
- net USB_DP_3V3: track 0.00 -> 9.96 mm
- net USB_DP_5V: track 0.00 -> 7.65 mm
- net USB_DM_5V: track 0.00 -> 5.68 mm
- added copper zone on layer 16, net 3.3V
Other:
- board size 67 x 20.3 mm -> 51.7 x 22.8 mm

Commit message: updates
Parts:
- added C12: UWD0J560MCL1GS, 56uF_Cap_6.3v:PCAP_5X5.8-ELECT
- added C13, C16: 1.0uF, SparkFun-Capacitors:0603
- added C14, C15: 0.1uF, SparkFun-Capacitors:0603
- added C17: 4.7uF, SparkFun-Capacitors:0603
- added R5: 1k, SparkFun-Resistors:0603
- added RESET: (no value), DiscreteComponents:SW_2512
- moved C8 37.6 mm to (53.3, 26.2), turned to 0 degrees
- moved U5 35.3 mm to (53.6, 23.1), turned to 90 degrees
- moved R1 34.1 mm to (56.6, 20.6), turned to 90 degrees
- moved C9 33.3 mm to (53.6, 19.6), turned to 180 degrees
- moved L1 30.8 mm to (49.3, 23.1), turned to 90 degrees
- moved U3 26.5 mm to (65.8, -10.4)
- moved U4 26.5 mm to (65.8, -4.32)
- moved R2 26.5 mm to (62.2, -10.4)
- moved R3 26.5 mm to (66.3, -7.37)
- moved R4 26.5 mm to (62.2, -4.32)
- moved R6 26.5 mm to (66.3, -1.27)
- moved C2 17.2 mm to (10.4, 13.2), turned to 90 degrees
- moved C11 13.6 mm to (40.9, 4.06), turned to 180 degrees
- moved C10 13.4 mm to (40.9, 12.7), turned to 180 degrees
- moved SV2 11.3 mm to (22.1, 6.86), turned to 90 degrees
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Connections:
- new net +3V3: R5.2
- net 3.3V: now also C12.1, C13.1, C14.1, C15.1, C16.1
- net CS: now also U1.14
- net DIO0: now also U1.19
- net GND: now also C12.2, C13.2, C14.2, C15.2, C16.2, C17.2, RESET.1
- net NRST: now also C17.1, R5.1, RESET.2
- net RST: now also U1.18
Routing:
- net USB_DM_3V3: track 17.0 -> 2.35 mm, vias 2 -> 0
- net USB_DP_3V3: track 9.96 -> 2.35 mm
- net 5V: track 13.6 -> 19.9 mm
- net USB_DP_5V: track 7.65 -> 3.09 mm
- net EN: track 0.00 -> 4.13 mm
- net N$2: track 0.00 -> 3.11 mm
- net USB_DM_5V: track 5.68 -> 3.09 mm
- net 3.3V: track 30.6 -> 33.1 mm
- added copper zone on layer 1, net 3.3V
Other:
- board size 51.7 x 22.8 mm -> 59.4 x 27.9 mm

Commit message: Finished Initial Routing
Parts:
- removed R2, R3, R4, R6: 10k, SparkFun-Resistors:0603
- removed U3, U4: BSS138, BSS138:SOT-23-3L
- added C18: 0.1uF, SparkFun-Capacitors:0603
- added CR1: USBLC6-2SC6, ESD_Protection:SOT23-6L
- added J2, J3: (no value), SparkFun-Connectors:1X03
- moved RESET 25.2 mm to (22.9, 12.6), turned to 270 degrees
- moved C17 24.6 mm to (22.9, 13.3), turned to 90 degrees
- moved SV2 23.8 mm to (45.5, 2.41), turned to 180 degrees
- moved R5 20.0 mm to (24.8, 13.3), flipped to the bottom
- moved C11 16.7 mm to (28.4, 15.2), turned to 0 degrees
- moved C10 13.9 mm to (28.4, 6.60), turned to 0 degrees
- moved C3 12.0 mm to (41.9, 9.65)
- moved C16 11.9 mm to (38.9, 14.0), turned to 0 degrees
- moved Y1 11.2 mm to (29.2, 10.9), turned to 90 degrees
- moved C15 9.54 mm to (38.9, 12.2), turned to 180 degrees
- moved C1 8.36 mm to (40.1, 9.65), turned to 270 degrees
- moved U1 7.52 mm to (38.4, 10.4), turned to 0 degrees
- moved C6 6.86 mm to (32.8, 18.0)
- moved C7 6.61 mm to (34.5, 18.0)
- moved C4 4.75 mm to (37.6, 8.64)
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Connections:
- removed net +3V3: R5.2
- removed net SPI_MOSI: U1.17
- removed net USB_DM_5V: J1.2, R6.2, U4.3
- removed net USB_DP_5V: J1.3, R3.2, U3.3
- new net USB_DM: CR1.4, J1.2
- new net USB_DP: CR1.6, J1.3
- net 3.3V: now also C18.1, CR1.5, J3.1, J3.2, J3.3, R5.2; no longer R2.2, R4.2, U3.1, U4.1
- net 5V: no longer R3.1, R6.1
- net GND: now also C18.2, CR1.2, J2.1, J2.2, J2.3
- net SPI1_MOSI: now also U1.17
- net USB_DM_3V3: now also CR1.3; no longer R4.1, U4.2
- net USB_DP_3V3: now also CR1.1; no longer R2.1, U3.2
Routing:
- net 3.3V: track 33.1 -> 135.0 mm, vias 3 -> 6
- net RST: track 0.00 -> 55.9 mm
- net SPI1_SCK: track 0.00 -> 52.4 mm, vias 0 -> 2
- net SPI1_MOSI: track 0.00 -> 52.0 mm
- net SPI1_MISO: track 0.00 -> 50.5 mm
- net CS: track 0.00 -> 50.2 mm, vias 0 -> 2
- net NRST: track 0.00 -> 48.4 mm, vias 0 -> 2
- net DIO0: track 0.00 -> 38.4 mm
- net GND: track 0.00 -> 37.5 mm, vias 0 -> 23
- net SWDIO: track 0.00 -> 18.6 mm, vias 0 -> 1
- net SWCLK: track 0.00 -> 15.8 mm, vias 0 -> 1
- net USB_DM: track 0.00 -> 7.89 mm
- net USB_DP: track 0.00 -> 7.83 mm
- net OSC_IN: track 0.00 -> 7.79 mm
- net OSC_OUT: track 0.00 -> 7.78 mm
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- added copper zone on layer 1, net N$3
- added copper zone on layer 16, net N$4
- added copper zone on layer 16, net N$5
Other:
- board text added: "MARS Base Station v1 2/3/2020 Jacob Bobson"
